File: digital_pot.sch (KiCad schematic (older format))
At the start: 5 parts

Commit message: Praca nad sch, dodana sekcja zasilania i karta sd
Parts:
- added C? (x34): 100n, symbol Device:C
- added R? (x10): R, symbol Device:R
- added U? (x21): ADA4898-3, Package_SO:SOIC-8-1EP_3.9x4.9mm_P1.27mm_EP2.41x3.81mm, symbol Amplifier_Operational:ADA4898-3
Connections:
- net input_voltage is gone; now on net +5V: U?.7 (PA1), U?.7 (PA1), U?.7 (PA1), U?.7 (PA1), U?.7 (PA1), U?.8 (PA0), U?.8 (PA0), U?.8 (PA0), U?.8 (PA0), U?.8 (PA0)
- net GND: now also C?.1, C?.1, C?.1, C?.1, C?.1, C?.1, C?.1, C?.1, C?.1, C?.1; no longer U?.10 (PB0), U?.10 (PB0), U?.10 (PB0), U?.10 (PB0), U?.10 (PB0), U?.5 (PB1), U?.5 (PB1), U?.5 (PB1), U?.5 (PB1), U?.5 (PB1)
- net B1: now reaches U?.6 (PW1)
- net B1: now also U?.12 (+)
- net A1: now reaches U?.9 (PW0)
- net A1: now also U?.5 (+)
- net B3: now reaches U?.6 (PW1)
- net B3: now also U?.12 (+)
- net A3: now reaches U?.9 (PW0)
- net A3: now also U?.5 (+)
- net B4: now reaches U?.6 (PW1)
- net B4: now also U?.12 (+)
- net A4: now reaches U?.9 (PW0)
- net A4: now also U?.5 (+)
- net B5: now reaches U?.6 (PW1)
- net B5: now also U?.12 (+)
- net A5: now reaches U?.9 (PW0)
- net A5: now also U?.5 (+)
- net B2: now reaches U?.6 (PW1)
- net B2: now also U?.12 (+)
- net A2: now reaches U?.9 (PW0)
- net A2: now also U?.5 (+)
- net VCC renamed +5V
- net +5V: now also C?.1, C?.1, C?.1, C?.1, C?.1, C?.1, C?.2, C?.2, C?.2, C?.2, C?.2, C?.2, C?.2, C?.2, C?.2, C?.2, C?.2, C?.2, C?.2, C?.2, C?.2, C?.2, U?.4 (V+), U?.4 (V+), U?.4 (V+), U?.4 (V+), U?.4 (V+), U?.4 (V+)
- new net: R?.1, R?.1, U?.10 (+) (x5)
- new net: R?.2, U?.6 (-), U?.7 (x5)
- new net: R?.2, U?.13 (-), U?.14 (x5)
- new net GNDA: C?.1, C?.1, C?.1, C?.1, C?.1, C?.1, C?.1, C?.1, C?.1, C?.1, C?.1, C?.1, C?.1, C?.1, C?.1, C?.1, C?.1, C?.1, C?.2, C?.2, C?.2, C?.2, C?.2, C?.2, C?.2, C?.2, C?.2, C?.2, C?.2, C?.2, C?.2, C?.2, C?.2, C?.2, C?.2, C?.2, U?.1 (~PD1), U?.1 (~PD1), U?.1 (~PD1), U?.1 (~PD1), U?.1 (~PD1), U?.1 (~PD1), U?.10 (PB0), U?.10 (PB0), U?.10 (PB0), U?.10 (PB0), U?.10 (PB0), U?.11 (V-), U?.11 (V-), U?.11 (V-), U?.11 (V-), U?.11 (V-), U?.11 (V-), U?.2 (~PD2), U?.2 (~PD2), U?.2 (~PD2), U?.2 (~PD2), U?.2 (~PD2), U?.2 (~PD2), U?.3 (~PD3), U?.3 (~PD3), U?.3 (~PD3), U?.3 (~PD3), U?.3 (~PD3), U?.3 (~PD3), U?.5 (PB1), U?.5 (PB1), U?.5 (PB1), U?.5 (PB1), U?.5 (PB1)
- new net OUT1: U?.8, U?.9 (-)
- new net OUT2: U?.8, U?.9 (-)
- new net OUT3: U?.8, U?.9 (-)
- new net OUT4: U?.8, U?.9 (-)
- new net OUT5: U?.8, U?.9 (-)
Other:
- note added: "amplifiers capacitor bank\n"
- note added: "digital pot capacitor bank\n"
- note added: "internal pull-up, but do not leave floating"
- note removed: "internal pull-up, do not leave floating"
- moved on the sheet: U?

Commit message: dalsza praca nad sch, przypisanie pinów
Parts:
- added C? (x8): 100n, symbol Device:C
- added R? (x6): R, symbol Device:R
- added U? (x3): MCP42050, symbol Potentiometer_Digital:MCP42050
- added U? (x11): ADA4898-3, Package_SO:SOIC-8-1EP_3.9x4.9mm_P1.27mm_EP2.41x3.81mm, symbol Amplifier_Operational:ADA4898-3
Connections:
- net +5V: now also C?.1, C?.1, C?.2, C?.2, U?.14 (VDD), U?.14 (VDD), U?.14 (VDD), U?.4 (V+), U?.4 (V+), U?.7 (PA1), U?.7 (PA1), U?.7 (PA1), U?.8 (PA0), U?.8 (PA0), U?.8 (PA0)
- net CS: now also U?.1 (~CS), U?.1 (~CS), U?.1 (~CS)
- net GND: now also U?.4 (VSS), U?.4 (VSS), U?.4 (VSS)
- net GNDA: now also C?.1, C?.1, C?.1, C?.1, C?.1, C?.1, C?.2, C?.2, C?.2, C?.2, C?.2, C?.2, U?.1 (~PD1), U?.1 (~PD1), U?.10 (PB0), U?.10 (PB0), U?.10 (PB0), U?.11 (V-), U?.11 (V-), U?.2 (~PD2), U?.2 (~PD2), U?.3 (~PD3), U?.3 (~PD3), U?.5 (PB1), U?.5 (PB1), U?.5 (PB1)
- net RST: now also U?.11 (~RS), U?.11 (~RS), U?.11 (~RS)
- net SCK: now also U?.2 (SCK), U?.2 (SCK), U?.2 (SCK)
- net SHDN: now also U?.12 (~SHDN), U?.12 (~SHDN), U?.12 (~SHDN)
- net at U?.13 (SO): now also U?.3 (SI)
- new net: U?.13 (SO), U?.3 (SI) (x2)
- new net: R?.1, R?.1, U?.10 (+) (x3)
- new net: R?.2, U?.13 (-), U?.14 (x3)
- new net: R?.2, U?.6 (-), U?.7 (x3)
- new net A6: U?.5 (+), U?.9 (PW0)
- new net A7: U?.5 (+), U?.9 (PW0)
- new net A8: U?.5 (+), U?.9 (PW0)
- new net B6: U?.12 (+), U?.6 (PW1)
- new net B7: U?.12 (+), U?.6 (PW1)
- new net B8: U?.12 (+), U?.6 (PW1)
- new net OUT6: U?.8, U?.9 (-)
- new net OUT7: U?.8, U?.9 (-)
- new net OUT8: U?.8, U?.9 (-)
- no-connect marks 0 -> 1
Other:
- moved on the sheet: C?, U?C
